Commit message: Adressed some changes
Calibrated tags, fixed axis, modified model so it's smaller, removed unnecesary files

File: ca_description/urdf/create_base.xacro (robot description, xacro)
@@ -42,5 +42,7 @@
       <origin xyz="0 -0.04 0.13" rpy="0 0 0"/>
     </xacro:imu_sensor>
-    <xacro:april_tag/>
+    <xacro:april_tag>
+      <origin xyz="0 0 0.25" rpy="0 0 1.577" />
+    </xacro:april_tag>
     <xacro:create_wheel prefix="left" y_offset="${wheel_separation / 2}" wheel_radius="${wheel_radius}" wheel_width="${wheel_width}"/>
     <xacro:create_wheel prefix="right" y_offset="${wheel_separation / -2}" wheel_radius="${wheel_radius}" wheel_width="${wheel_width}"/>

File: ca_description/urdf/sensors/apriltag.xacro (robot description, xacro)
@@ -1,9 +1,8 @@
 <?xml version="1.0"?>
 <robot xmlns:xacro="http://ros.org/wiki/xacro">
-    <xacro:macro name="april_tag">
+    <xacro:macro name="april_tag" params="*origin">
         <xacro:property name="april_tag_offset_z" value="0.25"/>
         <link name="april_tag_link">
             <visual>
-                <origin xyz="0 0 0" rpy="0 0 0" />
                 <geometry>
                     <box size="0.5 0.5 0.01"/>
@@ -12,8 +11,7 @@
         </link>
         <joint name="april_tag_joint" type="fixed">
-            <origin xyz="0 0 ${april_tag_offset_z}" rpy="0 0 0" />
+            <xacro:insert_block name="origin" />
             <parent link="base_link" />
             <child link="april_tag_link" />
-            <axis xyz="1 0 0"/>
         </joint>
         <!---->

Commit message: Add roscontrol

File: ca_description/urdf/create_base.xacro (robot description, xacro)
@@ -80,4 +80,24 @@
     <!-- Simulation sensors -->
     <xacro:sim_create_base/>
+    <transmission name="transmission">
+      <type>transmission_interface/SimpleTransmission</type>
+    <joint name="wheel_left_joint">
+      <hardwareInterface>hardware_interface/VelocityJointInterface</hardwareInterface>
+    </joint>
+    <actuator name="left_wheel_motor">
+      <hardwareInterface>hardware_interface/VelocityJointInterface</hardwareInterface>
+      <mechanicalReduction>1</mechanicalReduction>
+    </actuator>
+   </transmission>
+    <transmission name="transmission">
+      <type>transmission_interface/SimpleTransmission</type>
+    <joint name="wheel_right_joint">
+      <hardwareInterface>hardware_interface/VelocityJointInterface</hardwareInterface>
+    </joint>
+    <actuator name="right_wheel_motor">
+      <hardwareInterface>hardware_interface/VelocityJointInterface</hardwareInterface>
+      <mechanicalReduction>1</mechanicalReduction>
+    </actuator>
+   </transmission>
   </xacro:macro>
 </robot>

File: ca_description/urdf/create_base_gazebo.xacro (robot description, xacro)
@@ -3,25 +3,36 @@
   <xacro:macro name="sim_create_base">
     <gazebo>
+      <xacro:arg name="enable_ros_control" default="False"/>
       <!-- Diff-drive controller -->
-      <plugin name="differential_drive_controller" filename="libgazebo_ros_diff_drive.so">
-        <alwaysOn>true</alwaysOn>
-        <rosDebugLevel>na</rosDebugLevel>
-        <updateRate>30</updateRate>
-        <leftJoint>wheel_left_joint</leftJoint>
-        <rightJoint>wheel_right_joint</rightJoint>
-        <wheelSeparation>${wheel_separation}</wheelSeparation>
-        <wheelDiameter>${wheel_radius * 2}</wheelDiameter>
-        <wheelTorque>0.5</wheelTorque>
-        <wheelAcceleration>0.5</wheelAcceleration>
-        <commandTopic>cmd_vel</commandTopic>
-        <odometryTopic>odom</odometryTopic>
-        <odometryFrame>odom</odometryFrame>
-        <robotBaseFrame>base_footprint</robotBaseFrame>
-        <publishWheelTF>true</publishWheelTF>
-        <publishOdomTF>true</publishOdomTF>
-        <publishWheelJointState>true</publishWheelJointState>
-        <odometrySource>world</odometrySource>
-        <publishTf>true</publishTf>
+      <xacro:unless value="$(arg enable_ros_control)">
+        <plugin name="differential_drive_controller" filename="libgazebo_ros_diff_drive.so">
+          <alwaysOn>true</alwaysOn>
+          <rosDebugLevel>na</rosDebugLevel>
+          <updateRate>30</updateRate>
+          <leftJoint>wheel_left_joint</leftJoint>
+          <rightJoint>wheel_right_joint</rightJoint>
+          <wheelSeparation>${wheel_separation}</wheelSeparation>
+          <wheelDiameter>${wheel_radius * 2}</wheelDiameter>
+          <wheelTorque>0.5</wheelTorque>
+          <wheelAcceleration>0.5</wheelAcceleration>
+          <commandTopic>cmd_vel</commandTopic>
+          <odometryTopic>odom</odometryTopic>
+          <odometryFrame>odom</odometryFrame>
+          <robotBaseFrame>base_footprint</robotBaseFrame>
+          <publishWheelTF>true</publishWheelTF>
+          <publishOdomTF>true</publishOdomTF>
+          <publishWheelJointState>true</publishWheelJointState>
+          <odometrySource>world</odometrySource>
+          <publishTf>true</publishTf>
+        </plugin>
+    </xacro:unless>
+      <!-- ros_control plugin -->
+      <xacro:if value="$(arg enable_ros_control)">
+      <plugin name="gazebo_ros_control" filename="libgazebo_ros_control.so">
+        <robotNamespace>${robot_name}</robotNamespace>
+        <robotParam>robot_description</robotParam>
+        <robotSimType>gazebo_ros_control/DefaultRobotHWSim</robotSimType>
       </plugin>
+      </xacro:if>
       <!-- Ground truth -->
       <plugin name="p3d_base_controller" filename="libgazebo_ros_p3d.so">
